Commit message: add umi_moveit_config package

File: realsense_aruco_ws/src/umi_description/urdf/umi.xacro (robot description, xacro)
@@ -86,3 +86,9 @@
         <axis xyz="-1 0 0"/>
     </joint>
+    <link name="tool_link" />
+    <joint name="tool_link_2_umi_link" type="fixed">
+        <parent link="hand_link" />
+        <child link="tool_link" />
+        <origin rpy="0 0 0" xyz="0 0.01105 0.2" />
+    </joint>
 </robot>

Commit message: update umi gripper urdf (offset)

File: realsense_aruco_ws/src/umi_description/urdf/umi.xacro (robot description, xacro)
@@ -75,5 +75,5 @@
         <parent link="hand_link" />
         <child link="left_finger_link" />
-        <origin xyz="0 0.01105 0.108" rpy="0 0 0" />
+        <origin xyz="0 -0.01105 0.108" rpy="0 0 0" />
         <limit effort="100.0" lower="-0.04" upper="0" velocity="0.5"/>
         <axis xyz="1 0 0"/>
@@ -82,5 +82,5 @@
         <parent link="hand_link" />
         <child link="right_finger_link" />
-        <origin xyz="0 0.01105 0.108" rpy="0 0 0" />
+        <origin xyz="0 -0.01105 0.108" rpy="0 0 0" />
         <limit effort="100.0" lower="-0.04" upper="0" velocity="0.5"/>
         <axis xyz="-1 0 0"/>

Commit message: update umi.xacro

File: realsense_aruco_ws/src/umi_description/urdf/umi.xacro (robot description, xacro)
@@ -90,5 +90,5 @@
         <parent link="hand_link" />
         <child link="tool_link" />
-        <origin rpy="0 0 0" xyz="0 0.01105 0.2" />
+        <origin rpy="0 0 0" xyz="0 -0.01105 0.2" />
     </joint>
 </robot>

Commit message: add umi_control_from_moveit ros node

File: realsense_aruco_ws/src/umi_description/urdf/umi.xacro (robot description, xacro)
@@ -82,4 +82,5 @@
         <parent link="hand_link" />
         <child link="right_finger_link" />
+        <mimic joint="left_finger_joint" multiplier="1" offset="0" />
         <origin xyz="0 -0.01105 0.108" rpy="0 0 0" />
         <limit effort="100.0" lower="-0.04" upper="0" velocity="0.5"/>

Commit message: switch all interface to simulation

File: realsense_aruco_ws/src/umi_description/urdf/umi.xacro (robot description, xacro)
@@ -19,5 +19,5 @@
         <origin xyz="0 0 -0" rpy="0 0 0 " />
         <geometry>
-          <mesh filename="package://umi_description/meshes/hand.dae"/>
+          <mesh filename="package://umi_description/meshes/gripper_gopro.dae"/>
         </geometry>
       </visual>
@@ -25,5 +25,5 @@
         <origin xyz="0 0 0" rpy="0 0 0" />
         <geometry>
-          <mesh filename="package://umi_description/meshes/hand.STL" />
+          <mesh filename="package://umi_description/meshes/gripper_gopro.STL" />
         </geometry>
       </collision>
