Commit message: fix umi_control bugs

File: sim2sim_o3de_ws/src/umi_moveit_config/config/umi.ros2_control.xacro (robot description, xacro)
@@ -50,15 +50,15 @@
                 <state_interface name="velocity"/>
             </joint>
-            <joint name="dh_finger_joint1">
+            <joint name="left_finger_joint">
                 <command_interface name="position"/>
                 <state_interface name="position">
-                  <param name="initial_value">${initial_positions['dh_finger_joint1']}</param>
+                  <param name="initial_value">${initial_positions['left_finger_joint']}</param>
                 </state_interface>
                 <state_interface name="velocity"/>
             </joint>
-            <joint name="dh_finger_joint2">
+            <joint name="right_finger_joint">
                 <command_interface name="position"/>
                 <state_interface name="position">
-                  <param name="initial_value">${initial_positions['dh_finger_joint2']}</param>
+                  <param name="initial_value">${initial_positions['right_finger_joint']}</param>
                 </state_interface>
                 <state_interface name="velocity"/>
